Commit message: add autolauncher and default.rviz

File: src/swarm_sim_pkg/swarm_sim/assets/models/x500_sensors.sdf.xacro (robot description, xacro)
@@ -40,4 +40,7 @@
         <material><ambient>1 0 0 1</ambient><diffuse>1 0 0 1</diffuse></material>
       </visual>
+      <collision name="collision">
+        <geometry><box><size>0.02 0.05 0.02</size></box></geometry>
+      </collision>
       <sensor name="camera" type="camera">
         <camera>
@@ -69,4 +72,7 @@
         <material><ambient>1 1 0 1</ambient><diffuse>1 1 0 1</diffuse></material>
       </visual>
+      <collision name="collision">
+        <geometry><box><size>0.02 0.05 0.02</size></box></geometry>
+      </collision>
       <sensor name="down_camera" type="camera">
         <camera>

Commit message: fix lidar imu plugins

File: src/swarm_sim_pkg/swarm_sim/assets/models/x500_sensors.sdf.xacro (robot description, xacro)
@@ -1,10 +1,97 @@
-<?xml version="1.0" ?>
-<sdf version="1.9" xmlns:xacro="http://ros.org/wiki/xacro">
+<?xml version="1.0" encoding="UTF-8"?>
+<sdf version='1.9' xmlns:xacro="http://ros.org/wiki/xacro">
   <xacro:arg name="namespace" default="uav_0"/>
   <model name="$(arg namespace)">
-    <include merge="true">
-      <uri>https://fuel.gazebosim.org/1.0/PX4/models/x500</uri>
-    </include>
-    <!-- Velocity Control with Namespaced Topic -->
+    <pose>0 0 .24 0 0 0</pose>
+    <self_collide>false</self_collide>
+    <static>false</static>
+    <link name="base_link">
+      <inertial>
+        <mass>2.0</mass>
+        <inertia>
+          <ixx>0.02166666666666667</ixx>
+          <ixy>0</ixy>
+          <ixz>0</ixz>
+          <iyy>0.02166666666666667</iyy>
+          <iyz>0</iyz>
+          <izz>0.04000000000000001</izz>
+        </inertia>
+      </inertial>
+      <gravity>true</gravity>
+      <velocity_decay />
+      <!-- Frame Visual -->
+      <visual name="base_link_visual">
+        <pose>0 0 .025 0 0 3.141592654</pose>
+        <geometry>
+          <mesh>
+            <scale>1 1 1</scale>
+            <uri>file://$(find swarm_sim)/assets/PX4-gazebo-models/models/x500_base/meshes/NXP-HGD-CF.dae</uri>
+          </mesh>
+        </geometry>
+      </visual>
+      <!-- Motor Bases -->
+      <visual name="5010_motor_base_0">
+        <pose>0.174 0.174 .032 0 0 -.45</pose>
+        <geometry>
+          <mesh>
+            <scale>1 1 1</scale>
+            <uri>file://$(find swarm_sim)/assets/PX4-gazebo-models/models/x500_base/meshes/5010Base.dae</uri>
+          </mesh>
+        </geometry>
+      </visual>
+      <visual name="5010_motor_base_1">
+        <pose>-0.174 0.174 .032 0 0 -.45</pose>
+        <geometry>
+          <mesh>
+            <scale>1 1 1</scale>
+            <uri>file://$(find swarm_sim)/assets/PX4-gazebo-models/models/x500_base/meshes/5010Base.dae</uri>
+          </mesh>
+        </geometry>
+      </visual>
+      <visual name="5010_motor_base_2">
+        <pose>0.174 -0.174 .032 0 0 -.45</pose>
+        <geometry>
+          <mesh>
+            <scale>1 1 1</scale>
+            <uri>file://$(find swarm_sim)/assets/PX4-gazebo-models/models/x500_base/meshes/5010Base.dae</uri>
+          </mesh>
+        </geometry>
+      </visual>
+      <visual name="5010_motor_base_3">
+        <pose>-0.174 -0.174 .032 0 0 -.45</pose>
+        <geometry>
+          <mesh>
+            <scale>1 1 1</scale>
+            <uri>file://$(find swarm_sim)/assets/PX4-gazebo-models/models/x500_base/meshes/5010Base.dae</uri>
+          </mesh>
+        </geometry>
+      </visual>
+      <!-- Collisions -->
+      <collision name="base_link_collision_0">
+        <pose>0 0 .007 0 0 0</pose>
+        <geometry>
+          <box>
+            <size>0.35355 0.35355 0.05</size>
+          </box>
+        </geometry>
+      </collision>
+      <collision name="base_link_collision_1">
+        <pose>0 -0.098 -.123 -0.35 0 0</pose>
+        <geometry><box><size>0.015 0.015 0.21</size></box></geometry>
+      </collision>
+      <collision name="base_link_collision_2">
+        <pose>0 0.098 -.123 0.35 0 0</pose>
+        <geometry><box><size>0.015 0.015 0.21</size></box></geometry>
+      </collision>
+      <collision name="base_link_collision_3">
+        <pose>0 -0.132 -.2195 0 0 0</pose>
+        <geometry><box><size>0.25 0.015 0.015</size></box></geometry>
+      </collision>
+      <collision name="base_link_collision_4">
+        <pose>0 0.132 -.2195 0 0 0</pose>
+        <geometry><box><size>0.25 0.015 0.015</size></box></geometry>
+      </collision>
+    </link>
+    <!-- Velocity Control -->
     <plugin
       filename="gz-sim-velocity-control-system"
@@ -13,89 +100,8 @@
       <topic>/model/$(arg namespace)/cmd_vel</topic>
     </plugin>
-    <plugin
-      filename="gz-sim-odometry-publisher-system"
-      name="gz::sim::systems::OdometryPublisher">
-      <odom_frame>world</odom_frame>
-      <robot_base_frame>base_link</robot_base_frame>
-      <dimensions>3</dimensions>
-    </plugin>
-    <!-- Broadcast TF for all links -->
-    <plugin
-      filename="gz-sim-pose-publisher-system"
-      name="gz::sim::systems::PosePublisher">
-      <publish_link_pose>true</publish_link_pose>
-      <publish_sensor_pose>true</publish_sensor_pose>
-      <publish_collision_pose>false</publish_collision_pose>
-      <publish_visual_pose>false</publish_visual_pose>
-      <publish_nested_model_pose>true</publish_nested_model_pose>
-      <use_pose_vector_msg>true</use_pose_vector_msg>
-      <static_publisher>true</static_publisher>
-      <static_update_frequency>1</static_update_frequency>
-    </plugin>
-    <!-- Camera (Fixed on base) -->
-    <link name="camera_link">
-      <pose relative_to="base_link">0.1 0 0.1 0 0 0</pose>
-      <visual name="visual">
-        <geometry><box><size>0.02 0.05 0.02</size></box></geometry>
-        <material><ambient>1 0 0 1</ambient><diffuse>1 0 0 1</diffuse></material>
-      </visual>
-      <collision name="collision">
-        <geometry><box><size>0.02 0.05 0.02</size></box></geometry>
-      </collision>
-      <sensor name="camera" type="camera">
-        <camera>
-          <horizontal_fov>1.047</horizontal_fov>
-          <image>
-            <width>640</width>
-            <height>480</height>
-          </image>
-          <clip>
-            <near>0.1</near>
-            <far>100</far>
-          </clip>
-        </camera>
-        <always_on>1</always_on>
-        <update_rate>30</update_rate>
-        <visualize>true</visualize>
-        <topic>/model/$(arg namespace)/camera/image_raw</topic>
-      </sensor>
-    </link>
-    <joint name="camera_joint" type="fixed">
-        <parent>base_link</parent>
-        <child>camera_link</child>
-    </joint>
-    <!-- Downward Camera -->
-    <link name="down_camera_link">
-      <pose relative_to="base_link">0 0 -0.05 0 1.5708 0</pose>
-      <visual name="visual">
-        <geometry><box><size>0.02 0.05 0.02</size></box></geometry>
-        <material><ambient>1 1 0 1</ambient><diffuse>1 1 0 1</diffuse></material>
-      </visual>
-      <collision name="collision">
-        <geometry><box><size>0.02 0.05 0.02</size></box></geometry>
-      </collision>
-      <sensor name="down_camera" type="camera">
-        <camera>
-          <horizontal_fov>1.047</horizontal_fov>
-          <image>
-            <width>640</width>
-            <height>480</height>
-          </image>
-          <clip>
-            <near>0.1</near>
-            <far>100</far>
-          </clip>
-        </camera>
-        <always_on>1</always_on>
-        <update_rate>30</update_rate>
-        <visualize>true</visualize>
-        <topic>/model/$(arg namespace)/down_camera/image_raw</topic>
-      </sensor>
-    </link>
-    <joint name="down_camera_joint" type="fixed">
-        <parent>base_link</parent>
-        <child>down_camera_link</child>
-    </joint>
-    <!-- IMU Sensor -->
+    <!-- Plugins -->
+    <plugin filename="gz-sim-imu-system" name="gz::sim::systems::Imu"></plugin>
+    <!-- Custom Sensors Integration -->
+    <!-- IMU -->
     <link name="imu_link">
         <pose relative_to="base_link">0 0 0 0 0 0</pose>
@@ -103,7 +109,7 @@
             <mass>0.01</mass>
             <inertia>
-                <ixx>0.00001</ixx> <ixy>0</ixy> <ixz>0</ixz>
-                <iyy>0.00001</iyy> <iyz>0</iyz>
-                <izz>0.00001</izz>
+                <ixx>1e-5</ixx> <ixy>0</ixy> <ixz>0</ixz>
+                <iyy>1e-5</iyy> <iyz>0</iyz>
+                <izz>1e-5</izz>
             </inertia>
         </inertial>
@@ -119,37 +125,102 @@
         <child>imu_link</child>
     </joint>
-    <!-- 3D Lidar Top Link -->
+    <!-- Camera -->
+    <link name="camera_link">
+      <pose relative_to="base_link">0.1 0 0.05 0 0 0</pose>
+      <visual name="visual">
+        <geometry><box><size>0.02 0.05 0.02</size></box></geometry>
+        <material><ambient>1 0 0 1</ambient><diffuse>1 0 0 1</diffuse></material>
+      </visual>
+      <sensor name="camera" type="camera">
+        <camera>
+          <horizontal_fov>1.047</horizontal_fov>
+          <image><width>640</width><height>480</height></image>
+          <clip><near>0.1</near><far>100</far></clip>
+        </camera>
+        <always_on>1</always_on>
+        <update_rate>30</update_rate>
+        <visualize>true</visualize>
+        <topic>/model/$(arg namespace)/camera/image_raw</topic>
+      </sensor>
+    </link>
+    <joint name="camera_joint" type="fixed">
+        <parent>base_link</parent>
+        <child>camera_link</child>
+    </joint>
+    <!-- Downward Camera -->
+    <link name="down_camera_link">
+      <pose relative_to="base_link">0 0 -0.05 0 1.5708 0</pose>
+      <visual name="visual">
+        <geometry><box><size>0.02 0.05 0.02</size></box></geometry>
+        <material><ambient>0 1 0 1</ambient><diffuse>0 1 0 1</diffuse></material>
+      </visual>
+      <sensor name="down_camera" type="camera">
+        <camera>
+          <horizontal_fov>1.047</horizontal_fov>
+          <image><width>640</width><height>480</height></image>
+          <clip><near>0.1</near><far>100</far></clip>
+        </camera>
+        <always_on>1</always_on>
+        <update_rate>30</update_rate>
+        <visualize>true</visualize>
+        <topic>/model/$(arg namespace)/down_camera/image_raw</topic>
+      </sensor>
+    </link>
+    <joint name="down_camera_joint" type="fixed">
+        <parent>base_link</parent>
+        <child>down_camera_link</child>
+    </joint>
+    <!-- Sonar (Downward Lidar) -->
+    <link name="sonar_link">
+        <pose relative_to="base_link">0 0 -0.05 0 1.5708 0</pose>
+        <visual name="visual">
+            <geometry><box><size>0.02 0.02 0.01</size></box></geometry>
+            <material><ambient>0 1 0 1</ambient><diffuse>0 1 0 1</diffuse></material>
+        </visual>
+        <sensor name="sonar" type="gpu_lidar">
+            <topic>/model/$(arg namespace)/sonar/range</topic>
+            <update_rate>50</update_rate>
+            <visualize>true</visualize>
+            <ray>
+                <scan>
+                    <horizontal><samples>10</samples><resolution>1</resolution><min_angle>-0.15</min_angle><max_angle>0.15</max_angle></horizontal>
+                    <vertical><samples>10</samples><resolution>1</resolution><min_angle>-0.15</min_angle><max_angle>0.15</max_angle></vertical>
+                </scan>
+                <range><min>0.02</min><max>4.0</max><resolution>0.01</resolution></range>
+            </ray>
+        </sensor>
+    </link>
+    <joint name="sonar_joint" type="fixed">
+        <parent>base_link</parent>
+        <child>sonar_link</child>
+    </joint>
+    <!-- Spinning Lidar -->
     <link name="lidar_link">
-        <pose relative_to="base_link">0 0 0.25 0 0 0</pose> <!-- On top of X500 -->
+        <pose relative_to="base_link">0 0 0.08 0 0 0</pose>
+        <!-- Mount -->
+        <visual name="mount_stand">
+            <pose>0 0 -0.04 0 0 0</pose>
+            <geometry><cylinder><radius>0.02</radius><length>0.08</length></cylinder></geometry>
+            <material><ambient>0.1 0.1 0.1 1</ambient><diffuse>0.1 0.1 0.1 1</diffuse></material>
+        </visual>
+    </link>
+    <joint name="lidar_mount_joint" type="fixed">
+        <parent>base_link</parent>
+        <child>lidar_link</child>
+    </joint>
+    <link name="lidar_spin_link">
+        <pose relative_to="lidar_link">0 0 0 0 0 0</pose>
+        <inertial>
+            <mass>0.1</mass>
+            <inertia>
+                <ixx>0.0001</ixx> <ixy>0</ixy> <ixz>0</ixz>
+                <iyy>0.0001</iyy> <iyz>0</iyz>
+                <izz>0.0001</izz>
+            </inertia>
+        </inertial>
         <visual name="visual">
-            <geometry>
-                <cylinder>
-                    <radius>0.04</radius>
-                    <length>0.05</length>
-                </cylinder>
-            </geometry>
+            <geometry><cylinder><radius>0.035</radius><length>0.04</length></cylinder></geometry>
             <material><ambient>0 0 1 1</ambient><diffuse>0 0 1 1</diffuse></material>
         </visual>
-        <!-- Lidar Mount (Visual Stand) -->
-        <visual name="mount_visual">
-            <pose>0 0 -0.05 0 0 0</pose> <!-- Below the lidar -->
-            <geometry>
-                <cylinder>
-                    <radius>0.02</radius>
-                    <length>0.06</length>
-                </cylinder>
-            </geometry>
-            <material><ambient>0.2 0.2 0.2 1</ambient><diffuse>0.2 0.2 0.2 1</diffuse></material>
-        </visual>
-        <collision name="mount_collision">
-            <pose>0 0 -0.05 0 0 0</pose>
-            <geometry>
-                <cylinder>
-                    <radius>0.02</radius>
-                    <length>0.06</length>
-                </cylinder>
-            </geometry>
-        </collision>
-        <!-- 3D LiDAR -->
         <sensor name="lidar_3d" type="gpu_lidar">
           <topic>/model/$(arg namespace)/lidar/points</topic>
@@ -170,76 +241,79 @@
               </vertical>
             </scan>
-            <range>
-              <min>0.1</min>
-              <max>30.0</max>
-            </range>
+            <range><min>0.1</min><max>10.0</max></range>
           </ray>
-          <visualize>false</visualize>
+          <visualize>true</visualize>
           <always_on>1</always_on>
         </sensor>
     </link>
-    <joint name="lidar_joint" type="revolute">
-        <parent>base_link</parent>
-        <child>lidar_link</child>
+    <joint name="lidar_spin_joint" type="revolute">
+        <parent>lidar_link</parent>
+        <child>lidar_spin_link</child>
         <axis>
             <xyz>0 0 1</xyz>
-            <limit>
-                <lower>-10000000000000000</lower>
-                <upper>10000000000000000</upper>
-            </limit>
+            <limit><lower>-1e16</lower><upper>1e16</upper></limit>
         </axis>
     </joint>
-    <!-- Sonar (Simulated as Downward Lidar) -->
-    <link name="sonar_link">
-        <pose relative_to="base_link">0 0 -0.05 0 1.5708 0</pose> <!-- Bottom, pointing down (pitch 90) -->
-        <visual name="visual">
-            <geometry>
-                <box><size>0.02 0.02 0.01</size></box>
-            </geometry>
-            <material><ambient>0 1 0 1</ambient><diffuse>0 1 0 1</diffuse></material>
-        </visual>
-        <collision name="sonar_collision">
-            <geometry>
-                <box><size>0.02 0.02 0.01</size></box>
-            </geometry>
-        </collision>
-        <sensor name="sonar" type="gpu_lidar">
-            <topic>/model/$(arg namespace)/sonar/range</topic>
-            <update_rate>50</update_rate>
-            <visualize>true</visualize>
-            <ray>
-                <scan>
-                    <horizontal>
-                        <samples>10</samples>
-                        <resolution>1</resolution>
-                        <min_angle>-0.14835</min_angle>
-                        <max_angle>0.14835</max_angle>
-                    </horizontal>
-                    <vertical>
-                        <samples>10</samples>
-                        <resolution>1</resolution>
-                        <min_angle>-0.14835</min_angle>
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