Commit message: 3D to 2.5D with fixed altitude z

File: src/swarm_sim_pkg/swarm_sim/assets/models/x500.urdf.xacro (robot description, xacro)
@@ -71,10 +71,32 @@
     <origin xyz="0 0 0" rpy="0 0 0"/>
   </joint>
-  <!-- Sonar Link -->
-  <link name="$(arg namespace)/sonar_link"/>
-  <joint name="$(arg namespace)/sonar_joint" type="fixed">
+  <!-- Downward Lidar Link -->
+  <link name="$(arg namespace)/lidar_down_link">
+     <visual>
+      <geometry><cylinder length="0.02" radius="0.01"/></geometry>
+    </visual>
+  </link>
+  <joint name="$(arg namespace)/lidar_down_joint" type="fixed">
     <parent link="$(arg namespace)/base_link"/>
-    <child link="$(arg namespace)/sonar_link"/>
+    <child link="$(arg namespace)/lidar_down_link"/>
     <origin xyz="0 0 -0.05" rpy="0 1.5708 0"/>
   </joint>
+  <!-- Downward Lidar Sensor Frame (Matches Gazebo Frame ID) -->
+  <link name="$(arg namespace)/lidar_down_link/lidar_down"/>
+  <joint name="$(arg namespace)/lidar_down_sensor_joint" type="fixed">
+    <parent link="$(arg namespace)/lidar_down_link"/>
+    <child link="$(arg namespace)/lidar_down_link/lidar_down"/>
+    <origin xyz="0 0 0" rpy="0 0 0"/>
+  </joint>
+  <!-- GPS Link -->
+  <link name="$(arg namespace)/gps_link">
+    <visual>
+      <geometry><box size="0.01 0.01 0.01"/></geometry>
+    </visual>
+  </link>
+  <joint name="$(arg namespace)/gps_joint" type="fixed">
+    <parent link="$(arg namespace)/base_link"/>
+    <child link="$(arg namespace)/gps_link"/>
+    <origin xyz="0 0 0" rpy="0 0 0"/>
+  </joint>
 </robot>

File: src/swarm_sim_pkg/swarm_sim/assets/models/x500_sensors.sdf.xacro (robot description, xacro)
@@ -246,5 +246,5 @@
             <scan>
               <horizontal>
-                <samples>360</samples>
+                <samples>512</samples>
                 <resolution>1</resolution>
                 <min_angle>-3.14159</min_angle>
@@ -252,13 +252,19 @@
               </horizontal>
               <vertical>
-                <samples>16</samples>
+                <!-- Ouster OS1-64 Specs -->
+                <samples>64</samples>
                 <resolution>1</resolution>
-                <min_angle>-0.261799</min_angle>
-                <max_angle>0.261799</max_angle>
+                <min_angle>-0.2899</min_angle> <!-- -16.6 deg -->
+                <max_angle>0.2899</max_angle>  <!-- +16.6 deg -->
               </vertical>
             </scan>
-            <range><min>0.1</min><max>10.0</max></range>
+            <range><min>0.2</min><max>30.0</max></range>
+            <noise>
+              <type>gaussian</type>
+              <mean>0.0</mean>
+              <stddev>0.008</stddev>
+            </noise>
           </ray>
-          <visualize>true</visualize>
+          <visualize>false</visualize>
           <always_on>1</always_on>
         </sensor>
