Commit message: upgrade multi graph slam and fix lidar topic

File: install/swarm_sim/share/swarm_sim/assets/models/x500.urdf.xacro (robot description, xacro)
@@ -3,5 +3,5 @@
   <xacro:arg name="namespace" default="uav_0"/>
   <!-- Base Link -->
-  <link name="base_link">
+  <link name="$(arg namespace)/base_link">
     <visual>
       <origin xyz="0 0 0" rpy="0 0 0"/>
@@ -15,5 +15,5 @@
   </link>
   <!-- Lidar Link -->
-  <link name="lidar_link">
+  <link name="$(arg namespace)/lidar_link">
     <visual>
       <origin xyz="0 0 0" rpy="0 0 0"/>
@@ -21,57 +21,59 @@
     </visual>
   </link>
-  <joint name="lidar_joint" type="fixed">
-    <parent link="base_link"/>
-    <child link="lidar_link"/>
+  <joint name="$(arg namespace)/lidar_joint" type="fixed">
+    <parent link="$(arg namespace)/base_link"/>
+    <child link="$(arg namespace)/lidar_link"/>
     <origin xyz="0 0 0.08" rpy="0 0 0"/>
   </joint>
   <!-- Lidar Spin (Fixed for URDF Vis) -->
-  <link name="lidar_spin_link"/>
-  <joint name="lidar_spin_joint" type="fixed">
-    <parent link="lidar_link"/>
-    <child link="lidar_spin_link"/>
+  <link name="$(arg namespace)/lidar_spin_link"/>
+  <joint name="$(arg namespace)/lidar_spin_joint" type="fixed">
+    <parent link="$(arg namespace)/lidar_link"/>
+    <child link="$(arg namespace)/lidar_spin_link"/>
     <origin xyz="0 0 0" rpy="0 0 0"/>
   </joint>
-  <!-- Lidar Sensor Frame (Matches Gazebo Frame ID: uav_X/lidar_spin_link/lidar_3d) -->
-  <link name="lidar_spin_link/lidar_3d"/>
-  <joint name="lidar_sensor_joint" type="fixed">
-    <parent link="lidar_spin_link"/>
-    <child link="lidar_spin_link/lidar_3d"/>
-    <origin xyz="0 0 0" rpy="0 0 0"/> <!-- Sensor offset relative to spin link -->
+  <!-- Lidar Sensor Frame (Matches Gazebo Frame ID) -->
+  <!-- Note: Gazebo frame is uav_X/lidar_spin_link/lidar_3d.
+       If we prefix, we get uav_X/lidar_spin_link/lidar_3d because we want the exact string. -->
+  <link name="$(arg namespace)/lidar_spin_link/lidar_3d"/>
+  <joint name="$(arg namespace)/lidar_sensor_joint" type="fixed">
+    <parent link="$(arg namespace)/lidar_spin_link"/>
+    <child link="$(arg namespace)/lidar_spin_link/lidar_3d"/>
+    <origin xyz="0 0 0" rpy="0 0 0"/>
   </joint>
   <!-- Camera Link (Front) -->
-  <link name="camera_link">
+  <link name="$(arg namespace)/camera_link">
     <visual>
       <geometry><box size="0.02 0.05 0.02"/></geometry>
     </visual>
   </link>
-  <joint name="camera_joint" type="fixed">
-    <parent link="base_link"/>
-    <child link="camera_link"/>
+  <joint name="$(arg namespace)/camera_joint" type="fixed">
+    <parent link="$(arg namespace)/base_link"/>
+    <child link="$(arg namespace)/camera_link"/>
     <origin xyz="0.1 0 0.05" rpy="0 0 0"/>
   </joint>
   <!-- Down Camera Link -->
-  <link name="down_camera_link">
+  <link name="$(arg namespace)/down_camera_link">
      <visual>
       <geometry><box size="0.02 0.05 0.02"/></geometry>
     </visual>
   </link>
-  <joint name="down_camera_joint" type="fixed">
-    <parent link="base_link"/>
-    <child link="down_camera_link"/>
+  <joint name="$(arg namespace)/down_camera_joint" type="fixed">
+    <parent link="$(arg namespace)/base_link"/>
+    <child link="$(arg namespace)/down_camera_link"/>
     <origin xyz="0 0 -0.05" rpy="0 1.5708 0"/>
   </joint>
   <!-- IMU Link -->
-  <link name="imu_link"/>
-  <joint name="imu_joint" type="fixed">
-    <parent link="base_link"/>
-    <child link="imu_link"/>
+  <link name="$(arg namespace)/imu_link"/>
+  <joint name="$(arg namespace)/imu_joint" type="fixed">
+    <parent link="$(arg namespace)/base_link"/>
+    <child link="$(arg namespace)/imu_link"/>
     <origin xyz="0 0 0" rpy="0 0 0"/>
   </joint>
   <!-- Sonar Link -->
-  <link name="sonar_link"/>
-  <joint name="sonar_joint" type="fixed">
-    <parent link="base_link"/>
-    <child link="sonar_link"/>
+  <link name="$(arg namespace)/sonar_link"/>
+  <joint name="$(arg namespace)/sonar_joint" type="fixed">
+    <parent link="$(arg namespace)/base_link"/>
+    <child link="$(arg namespace)/sonar_link"/>
     <origin xyz="0 0 -0.05" rpy="0 1.5708 0"/>
   </joint>

File: install/swarm_sim/share/swarm_sim/assets/models/x500_sensors.sdf.xacro (robot description, xacro)
@@ -102,4 +102,11 @@
     <!-- Plugins -->
     <plugin filename="gz-sim-imu-system" name="gz::sim::systems::Imu"></plugin>
+    <plugin filename="gz-sim-odometry-publisher-system" name="gz::sim::systems::OdometryPublisher">
+      <odom_frame>world</odom_frame>
+      <robot_base_frame>base_link</robot_base_frame>
+      <odom_publish_frequency>50</odom_publish_frequency>
+      <topic>/model/$(arg namespace)/odometry</topic>
+      <dimensions>3</dimensions>
+    </plugin>
     <!-- Custom Sensors Integration -->
     <!-- IMU -->

File: src/swarm_sim_pkg/swarm_sim/assets/models/x500_sensors.sdf.xacro (robot description, xacro)
@@ -102,4 +102,11 @@
     <!-- Plugins -->
     <plugin filename="gz-sim-imu-system" name="gz::sim::systems::Imu"></plugin>
+    <plugin filename="gz-sim-odometry-publisher-system" name="gz::sim::systems::OdometryPublisher">
+      <odom_frame>world</odom_frame>
+      <robot_base_frame>$(arg namespace)/base_link</robot_base_frame>
+      <odom_publish_frequency>50</odom_publish_frequency>
+      <topic>/model/$(arg namespace)/odometry</topic>
+      <dimensions>3</dimensions>
+    </plugin>
     <!-- Custom Sensors Integration -->
     <!-- IMU -->
