Commit message: fix env RL"

File: install/swarm_sim/share/swarm_sim/assets/models/x500.urdf.xacro (robot description, xacro)
@@ -1,80 +1 @@
-<?xml version="1.0"?>
-<robot name="x500" xmlns:xacro="http://ros.org/wiki/xacro">
-  <xacro:arg name="namespace" default="uav_0"/>
-  <!-- Base Link -->
-  <link name="$(arg namespace)/base_link">
-    <visual>
-      <origin xyz="0 0 0" rpy="0 0 0"/>
-      <geometry>
-        <box size="0.4 0.4 0.1"/>
-      </geometry>
-      <material name="grey">
-        <color rgba="0.5 0.5 0.5 1.0"/>
-      </material>
-    </visual>
-  </link>
-  <!-- Lidar Link -->
-  <link name="$(arg namespace)/lidar_link">
-    <visual>
-      <origin xyz="0 0 0" rpy="0 0 0"/>
-      <geometry><cylinder length="0.08" radius="0.03"/></geometry>
-    </visual>
-  </link>
-  <joint name="$(arg namespace)/lidar_joint" type="fixed">
-    <parent link="$(arg namespace)/base_link"/>
-    <child link="$(arg namespace)/lidar_link"/>
-    <origin xyz="0 0 0.08" rpy="0 0 0"/>
-  </joint>
-  <!-- Lidar Spin (Fixed for URDF Vis) -->
-  <link name="$(arg namespace)/lidar_spin_link"/>
-  <joint name="$(arg namespace)/lidar_spin_joint" type="fixed">
-    <parent link="$(arg namespace)/lidar_link"/>
-    <child link="$(arg namespace)/lidar_spin_link"/>
-    <origin xyz="0 0 0" rpy="0 0 0"/>
-  </joint>
-  <!-- Lidar Sensor Frame (Matches Gazebo Frame ID) -->
-  <!-- Note: Gazebo frame is uav_X/lidar_spin_link/lidar_3d.
-       If we prefix, we get uav_X/lidar_spin_link/lidar_3d because we want the exact string. -->
-  <link name="$(arg namespace)/lidar_spin_link/lidar_3d"/>
-  <joint name="$(arg namespace)/lidar_sensor_joint" type="fixed">
-    <parent link="$(arg namespace)/lidar_spin_link"/>
-    <child link="$(arg namespace)/lidar_spin_link/lidar_3d"/>
-    <origin xyz="0 0 0" rpy="0 0 0"/>
-  </joint>
-  <!-- Camera Link (Front) -->
-  <link name="$(arg namespace)/camera_link">
-    <visual>
-      <geometry><box size="0.02 0.05 0.02"/></geometry>
-    </visual>
-  </link>
-  <joint name="$(arg namespace)/camera_joint" type="fixed">
-    <parent link="$(arg namespace)/base_link"/>
-    <child link="$(arg namespace)/camera_link"/>
-    <origin xyz="0.1 0 0.05" rpy="0 0 0"/>
-  </joint>
-  <!-- Down Camera Link -->
-  <link name="$(arg namespace)/down_camera_link">
-     <visual>
-      <geometry><box size="0.02 0.05 0.02"/></geometry>
-    </visual>
-  </link>
-  <joint name="$(arg namespace)/down_camera_joint" type="fixed">
-    <parent link="$(arg namespace)/base_link"/>
-    <child link="$(arg namespace)/down_camera_link"/>
-    <origin xyz="0 0 -0.05" rpy="0 1.5708 0"/>
-  </joint>
-  <!-- IMU Link -->
-  <link name="$(arg namespace)/imu_link"/>
-  <joint name="$(arg namespace)/imu_joint" type="fixed">
-    <parent link="$(arg namespace)/base_link"/>
-    <child link="$(arg namespace)/imu_link"/>
-    <origin xyz="0 0 0" rpy="0 0 0"/>
-  </joint>
-  <!-- Sonar Link -->
-  <link name="$(arg namespace)/sonar_link"/>
-  <joint name="$(arg namespace)/sonar_joint" type="fixed">
-    <parent link="$(arg namespace)/base_link"/>
-    <child link="$(arg namespace)/sonar_link"/>
-    <origin xyz="0 0 -0.05" rpy="0 1.5708 0"/>
-  </joint>
-</robot>
+/mnt/disk1/pgguedje/research/gazebo_ros2_vnc/build/swarm_sim/swarm_sim/assets/models/x500.urdf.xacro

File: install/swarm_sim/share/swarm_sim/assets/models/x500_sensors.sdf.xacro (robot description, xacro)
@@ -1,326 +1 @@
-<?xml version="1.0" encoding="UTF-8"?>
-<sdf version='1.9' xmlns:xacro="http://ros.org/wiki/xacro">
-  <xacro:arg name="namespace" default="uav_0"/>
-  <model name="$(arg namespace)">
-    <pose>0 0 .24 0 0 0</pose>
-    <self_collide>false</self_collide>
-    <static>false</static>
-    <link name="base_link">
-      <inertial>
-        <mass>2.0</mass>
-        <inertia>
-          <ixx>0.02166666666666667</ixx>
-          <ixy>0</ixy>
-          <ixz>0</ixz>
-          <iyy>0.02166666666666667</iyy>
-          <iyz>0</iyz>
-          <izz>0.04000000000000001</izz>
-        </inertia>
-      </inertial>
-      <gravity>true</gravity>
-      <velocity_decay />
-      <!-- Frame Visual -->
-      <visual name="base_link_visual">
-        <pose>0 0 .025 0 0 3.141592654</pose>
-        <geometry>
-          <mesh>
-            <scale>1 1 1</scale>
-            <uri>file://$(find swarm_sim)/assets/PX4-gazebo-models/models/x500_base/meshes/NXP-HGD-CF.dae</uri>
-          </mesh>
-        </geometry>
-      </visual>
-      <!-- Motor Bases -->
-      <visual name="5010_motor_base_0">
-        <pose>0.174 0.174 .032 0 0 -.45</pose>
-        <geometry>
-          <mesh>
-            <scale>1 1 1</scale>
-            <uri>file://$(find swarm_sim)/assets/PX4-gazebo-models/models/x500_base/meshes/5010Base.dae</uri>
-          </mesh>
-        </geometry>
-      </visual>
-      <visual name="5010_motor_base_1">
-        <pose>-0.174 0.174 .032 0 0 -.45</pose>
-        <geometry>
-          <mesh>
-            <scale>1 1 1</scale>
-            <uri>file://$(find swarm_sim)/assets/PX4-gazebo-models/models/x500_base/meshes/5010Base.dae</uri>
-          </mesh>
-        </geometry>
-      </visual>
-      <visual name="5010_motor_base_2">
-        <pose>0.174 -0.174 .032 0 0 -.45</pose>
-        <geometry>
-          <mesh>
-            <scale>1 1 1</scale>
-            <uri>file://$(find swarm_sim)/assets/PX4-gazebo-models/models/x500_base/meshes/5010Base.dae</uri>
-          </mesh>
-        </geometry>
-      </visual>
-      <visual name="5010_motor_base_3">
-        <pose>-0.174 -0.174 .032 0 0 -.45</pose>
-        <geometry>
-          <mesh>
-            <scale>1 1 1</scale>
-            <uri>file://$(find swarm_sim)/assets/PX4-gazebo-models/models/x500_base/meshes/5010Base.dae</uri>
-          </mesh>
-        </geometry>
-      </visual>
-      <!-- Collisions -->
-      <collision name="base_link_collision_0">
-        <pose>0 0 .007 0 0 0</pose>
-        <geometry>
-          <box>
-            <size>0.35355 0.35355 0.05</size>
-          </box>
-        </geometry>
-      </collision>
-      <collision name="base_link_collision_1">
-        <pose>0 -0.098 -.123 -0.35 0 0</pose>
-        <geometry><box><size>0.015 0.015 0.21</size></box></geometry>
-      </collision>
-      <collision name="base_link_collision_2">
-        <pose>0 0.098 -.123 0.35 0 0</pose>
-        <geometry><box><size>0.015 0.015 0.21</size></box></geometry>
-      </collision>
-      <collision name="base_link_collision_3">
-        <pose>0 -0.132 -.2195 0 0 0</pose>
-        <geometry><box><size>0.25 0.015 0.015</size></box></geometry>
-      </collision>
-      <collision name="base_link_collision_4">
-        <pose>0 0.132 -.2195 0 0 0</pose>
-        <geometry><box><size>0.25 0.015 0.015</size></box></geometry>
-      </collision>
-    </link>
-    <!-- Velocity Control -->
-    <plugin
-      filename="gz-sim-velocity-control-system"
-      name="gz::sim::systems::VelocityControl">
-      <link_name>base_link</link_name>
-      <topic>/model/$(arg namespace)/cmd_vel</topic>
-    </plugin>
-    <!-- Plugins -->
-    <plugin filename="gz-sim-imu-system" name="gz::sim::systems::Imu"></plugin>
-    <plugin filename="gz-sim-odometry-publisher-system" name="gz::sim::systems::OdometryPublisher">
-      <odom_frame>world</odom_frame>
-      <robot_base_frame>base_link</robot_base_frame>
-      <odom_publish_frequency>50</odom_publish_frequency>
-      <topic>/model/$(arg namespace)/odometry</topic>
-      <dimensions>3</dimensions>
-    </plugin>
-    <!-- Custom Sensors Integration -->
-    <!-- IMU -->
-    <link name="imu_link">
-        <pose relative_to="base_link">0 0 0 0 0 0</pose>
-        <inertial>
-            <mass>0.01</mass>
-            <inertia>
-                <ixx>1e-5</ixx> <ixy>0</ixy> <ixz>0</ixz>
-                <iyy>1e-5</iyy> <iyz>0</iyz>
-                <izz>1e-5</izz>
-            </inertia>
-        </inertial>
-        <sensor name="imu_sensor" type="imu">
-            <always_on>1</always_on>
-            <update_rate>100</update_rate>
-            <visualize>true</visualize>
-            <topic>/model/$(arg namespace)/imu</topic>
-        </sensor>
-    </link>
-    <joint name="imu_joint" type="fixed">
-        <parent>base_link</parent>
-        <child>imu_link</child>
-    </joint>
-    <!-- Camera -->
-    <link name="camera_link">
-      <pose relative_to="base_link">0.1 0 0.05 0 0 0</pose>
-      <visual name="visual">
-        <geometry><box><size>0.02 0.05 0.02</size></box></geometry>
-        <material><ambient>1 0 0 1</ambient><diffuse>1 0 0 1</diffuse></material>
-      </visual>
-      <sensor name="camera" type="camera">
-        <camera>
-          <horizontal_fov>1.047</horizontal_fov>
-          <image><width>640</width><height>480</height></image>
-          <clip><near>0.1</near><far>100</far></clip>
-        </camera>
-        <always_on>1</always_on>
-        <update_rate>30</update_rate>
-        <visualize>true</visualize>
-        <topic>/model/$(arg namespace)/camera/image_raw</topic>
-      </sensor>
-    </link>
-    <joint name="camera_joint" type="fixed">
-        <parent>base_link</parent>
-        <child>camera_link</child>
-    </joint>
-    <!-- Downward Camera -->
-    <link name="down_camera_link">
-      <pose relative_to="base_link">0 0 -0.05 0 1.5708 0</pose>
-      <visual name="visual">
-        <geometry><box><size>0.02 0.05 0.02</size></box></geometry>
-        <material><ambient>0 1 0 1</ambient><diffuse>0 1 0 1</diffuse></material>
-      </visual>
-      <sensor name="down_camera" type="camera">
-        <camera>
-          <horizontal_fov>1.047</horizontal_fov>
-          <image><width>640</width><height>480</height></image>
-          <clip><near>0.1</near><far>100</far></clip>
-        </camera>
-        <always_on>1</always_on>
-        <update_rate>30</update_rate>
-        <visualize>true</visualize>
-        <topic>/model/$(arg namespace)/down_camera/image_raw</topic>
-      </sensor>
-    </link>
-    <joint name="down_camera_joint" type="fixed">
-        <parent>base_link</parent>
-        <child>down_camera_link</child>
-    </joint>
-    <!-- Sonar (Downward Lidar) -->
-    <link name="sonar_link">
-        <pose relative_to="base_link">0 0 -0.05 0 1.5708 0</pose>
-        <visual name="visual">
-            <geometry><box><size>0.02 0.02 0.01</size></box></geometry>
-            <material><ambient>0 1 0 1</ambient><diffuse>0 1 0 1</diffuse></material>
-        </visual>
-        <sensor name="sonar" type="gpu_lidar">
-            <topic>/model/$(arg namespace)/sonar/range</topic>
-            <update_rate>50</update_rate>
-            <visualize>true</visualize>
-            <ray>
-                <scan>
-                    <horizontal><samples>10</samples><resolution>1</resolution><min_angle>-0.15</min_angle><max_angle>0.15</max_angle></horizontal>
-                    <vertical><samples>10</samples><resolution>1</resolution><min_angle>-0.15</min_angle><max_angle>0.15</max_angle></vertical>
-                </scan>
-                <range><min>0.02</min><max>4.0</max><resolution>0.01</resolution></range>
-            </ray>
-        </sensor>
-    </link>
-    <joint name="sonar_joint" type="fixed">
-        <parent>base_link</parent>
-        <child>sonar_link</child>
-    </joint>
-    <!-- Spinning Lidar -->
-    <link name="lidar_link">
-        <pose relative_to="base_link">0 0 0.08 0 0 0</pose>
-        <!-- Mount -->
-        <visual name="mount_stand">
-            <pose>0 0 -0.04 0 0 0</pose>
-            <geometry><cylinder><radius>0.02</radius><length>0.08</length></cylinder></geometry>
-            <material><ambient>0.1 0.1 0.1 1</ambient><diffuse>0.1 0.1 0.1 1</diffuse></material>
-        </visual>
-    </link>
-    <joint name="lidar_mount_joint" type="fixed">
-        <parent>base_link</parent>
-        <child>lidar_link</child>
-    </joint>
-    <link name="lidar_spin_link">
-        <pose relative_to="lidar_link">0 0 0 0 0 0</pose>
-        <inertial>
-            <mass>0.1</mass>
-            <inertia>
-                <ixx>0.0001</ixx> <ixy>0</ixy> <ixz>0</ixz>
-                <iyy>0.0001</iyy> <iyz>0</iyz>
-                <izz>0.0001</izz>
-            </inertia>
-        </inertial>
-        <visual name="visual">
-            <geometry><cylinder><radius>0.035</radius><length>0.04</length></cylinder></geometry>
-            <material><ambient>0 0 1 1</ambient><diffuse>0 0 1 1</diffuse></material>
-        </visual>
-        <sensor name="lidar_3d" type="gpu_lidar">
-          <topic>/model/$(arg namespace)/lidar/points</topic>
-          <update_rate>10</update_rate>
-          <ray>
-            <scan>
-              <horizontal>
-                <samples>360</samples>
-                <resolution>1</resolution>
-                <min_angle>-3.14159</min_angle>
-                <max_angle>3.14159</max_angle>
-              </horizontal>
-              <vertical>
-                <samples>16</samples>
-                <resolution>1</resolution>
-                <min_angle>-0.261799</min_angle>
-                <max_angle>0.261799</max_angle>
-              </vertical>
-            </scan>
-            <range><min>0.1</min><max>10.0</max></range>
-          </ray>
-          <visualize>true</visualize>
-          <always_on>1</always_on>
-        </sensor>
-    </link>
-    <joint name="lidar_spin_joint" type="revolute">
-        <parent>lidar_link</parent>
-        <child>lidar_spin_link</child>
-        <axis>
-            <xyz>0 0 1</xyz>
-            <limit><lower>-1e16</lower><upper>1e16</upper></limit>
-        </axis>
-    </joint>
-    <plugin filename="gz-sim-joint-controller-system" name="gz::sim::systems::JointController">
-      <joint_name>lidar_spin_joint</joint_name>
-      <initial_velocity>6.28</initial_velocity>
-    </plugin>
-    <!-- Propellers (Rotors) - Visual Only for now (to save physics complexity) -->
-    <!-- Rotor 0 -->
-    <link name="rotor_0">
-      <pose>0.174 -0.174 0.06 0 0 0</pose>
-      <visual name="rotor_0_visual">
-        <pose>-0.022 -0.146 -0.016 0 0 0</pose>
-        <geometry><mesh><scale>0.846 0.846 0.846</scale><uri>file://$(find swarm_sim)/assets/PX4-gazebo-models/models/x500_base/meshes/1345_prop_ccw.stl</uri></mesh></geometry>
-        <material><ambient>0.2 0.2 0.2 1</ambient><diffuse>0.2 0.2 0.2 1</diffuse></material>
-      </visual>
-      <visual name="rotor_0_bell">
-        <pose>0 0 -.032 0 0 0</pose>
-        <geometry><mesh><scale>1 1 1</scale><uri>file://$(find swarm_sim)/assets/PX4-gazebo-models/models/x500_base/meshes/5010Bell.dae</uri></mesh></geometry>
-      </visual>
-    </link>
-    <joint name="rotor_0_joint" type="fixed"><parent>base_link</parent><child>rotor_0</child></joint>
-    <!-- Rotor 1 -->
-    <link name="rotor_1">
-      <pose>-0.174 0.174 0.06 0 0 0</pose>
-      <visual name="rotor_1_visual">
-        <pose>-0.022 -0.146 -0.016 0 0 0</pose>
-        <geometry><mesh><scale>0.846 0.846 0.846</scale><uri>file://$(find swarm_sim)/assets/PX4-gazebo-models/models/x500_base/meshes/1345_prop_ccw.stl</uri></mesh></geometry>
-        <material><ambient>0.2 0.2 0.2 1</ambient><diffuse>0.2 0.2 0.2 1</diffuse></material>
-      </visual>
-      <visual name="rotor_1_bell">
-        <pose>0 0 -.032 0 0 0</pose>
-        <geometry><mesh><scale>1 1 1</scale><uri>file://$(find swarm_sim)/assets/PX4-gazebo-models/models/x500_base/meshes/5010Bell.dae</uri></mesh></geometry>
-      </visual>
-    </link>
-    <joint name="rotor_1_joint" type="fixed"><parent>base_link</parent><child>rotor_1</child></joint>
-    <!-- Rotor 2 -->
-    <link name="rotor_2">
-      <pose>0.174 0.174 0.06 0 0 0</pose>
-      <visual name="rotor_2_visual">
-        <pose>-0.022 -0.146 -0.016 0 0 0</pose>
-        <geometry><mesh><scale>0.846 0.846 0.846</scale><uri>file://$(find swarm_sim)/assets/PX4-gazebo-models/models/x500_base/meshes/1345_prop_cw.stl</uri></mesh></geometry>
-        <material><ambient>0.2 0.2 0.2 1</ambient><diffuse>0.2 0.2 0.2 1</diffuse></material>
-      </visual>
-      <visual name="rotor_2_bell">
-        <pose>0 0 -.032 0 0 0</pose>
-        <geometry><mesh><scale>1 1 1</scale><uri>file://$(find swarm_sim)/assets/PX4-gazebo-models/models/x500_base/meshes/5010Bell.dae</uri></mesh></geometry>
-      </visual>
-    </link>
-    <joint name="rotor_2_joint" type="fixed"><parent>base_link</parent><child>rotor_2</child></joint>
-    <!-- Rotor 3 -->
-    <link name="rotor_3">
-      <pose>-0.174 -0.174 0.06 0 0 0</pose>
-      <visual name="rotor_3_visual">
-        <pose>-0.022 -0.146 -0.016 0 0 0</pose>
-        <geometry><mesh><scale>0.846 0.846 0.846</scale><uri>file://$(find swarm_sim)/assets/PX4-gazebo-models/models/x500_base/meshes/1345_prop_cw.stl</uri></mesh></geometry>
-        <material><ambient>0.2 0.2 0.2 1</ambient><diffuse>0.2 0.2 0.2 1</diffuse></material>
-      </visual>
-      <visual name="rotor_3_bell">
-        <pose>0 0 -.032 0 0 0</pose>
-        <geometry><mesh><scale>1 1 1</scale><uri>file://$(find swarm_sim)/assets/PX4-gazebo-models/models/x500_base/meshes/5010Bell.dae</uri></mesh></geometry>
-      </visual>
-    </link>
-    <joint name="rotor_3_joint" type="fixed"><parent>base_link</parent><child>rotor_3</child></joint>
-  </model>
-</sdf>
+/mnt/disk1/pgguedje/research/gazebo_ros2_vnc/build/swarm_sim/swarm_sim/assets/models/x500_sensors.sdf.xacro

File: src/swarm_sim_pkg/swarm_sim/assets/models/x500_sensors.sdf.xacro (robot description, xacro)
@@ -178,27 +178,37 @@
         <child>down_camera_link</child>
     </joint>
-    <!-- Sonar (Downward Lidar) -->
-    <link name="sonar_link">
+    <!-- Downward Lidar (Mapping Scanner) -->
+    <link name="lidar_down_link">
         <pose relative_to="base_link">0 0 -0.05 0 1.5708 0</pose>
         <visual name="visual">
-            <geometry><box><size>0.02 0.02 0.01</size></box></geometry>
+            <geometry><cylinder><radius>0.01</radius><length>0.02</length></cylinder></geometry>
             <material><ambient>0 1 0 1</ambient><diffuse>0 1 0 1</diffuse></material>
         </visual>
-        <sensor name="sonar" type="gpu_lidar">
-            <topic>/model/$(arg namespace)/sonar/range</topic>
-            <update_rate>50</update_rate>
+        <sensor name="lidar_down" type="gpu_lidar">
+            <topic>/model/$(arg namespace)/lidar_down/points</topic>
+            <update_rate>20</update_rate>
             <visualize>true</visualize>
             <ray>
                 <scan>
-                    <horizontal><samples>10</samples><resolution>1</resolution><min_angle>-0.15</min_angle><max_angle>0.15</max_angle></horizontal>
-                    <vertical><samples>10</samples><resolution>1</resolution><min_angle>-0.15</min_angle><max_angle>0.15</max_angle></vertical>
+                    <horizontal>
+                        <samples>64</samples>
+                        <resolution>1</resolution>
+                        <min_angle>-0.785</min_angle> <!-- -45 deg -->
+                        <max_angle>0.785</max_angle>  <!-- +45 deg -->
+                    </horizontal>
+                    <vertical>
+                        <samples>64</samples>
+                        <resolution>1</resolution>
+                        <min_angle>-0.785</min_angle> <!-- -45 deg -->
+                        <max_angle>0.785</max_angle>  <!-- +45 deg -->
+                    </vertical>
                 </scan>
-                <range><min>0.02</min><max>4.0</max><resolution>0.01</resolution></range>
+                <range><min>0.1</min><max>15.0</max><resolution>0.02</resolution></range>
             </ray>
         </sensor>
     </link>
-    <joint name="sonar_joint" type="fixed">
-        <parent>base_link</parent>
-        <child>sonar_link</child>
+    <joint name="lidar_down_joint" type="fixed">
+        <parent>base_link</parent>
+        <child>lidar_down_link</child>
     </joint>
     <!-- Spinning Lidar -->
@@ -266,4 +276,23 @@
       <initial_velocity>6.28</initial_velocity>
     </plugin>
+    <!-- GPS Plugin -->
+    <plugin filename="gz-sim-navsat-system" name="gz::sim::systems::NavSat"></plugin>
+    <!-- GPS Sensor -->
+    <link name="gps_link">
+        <pose relative_to="base_link">0 0 0 0 0 0</pose>
+        <visual name="visual">
+            <geometry><box><size>0.01 0.01 0.01</size></box></geometry>
+            <material><ambient>0 0 0 1</ambient><diffuse>0 0 0 1</diffuse></material>
+        </visual>
+        <sensor name="navsat" type="navsat">
+            <always_on>1</always_on>
+            <update_rate>5</update_rate>
+            <topic>/model/$(arg namespace)/navsat</topic>
+        </sensor>
+    </link>
+    <joint name="gps_joint" type="fixed">
+        <parent>base_link</parent>
+        <child>gps_link</child>
+    </joint>
     <!-- Propellers (Rotors) - Visual Only for now (to save physics complexity) -->
     <!-- Rotor 0 -->
